Commit message: add camera on rover package

File: src/rover_arm_new_urdf/urdf/rover_arm_new_urdf.urdf (robot description, URDF)
Before this commit: robot rover_arm_new_urdf, 9 links, 8 joints
Links:
- added link camera_link, mass 0.001; visual box size=0.01 0.01 0.01
Joints:
- added joint camera_joint: type fixed, parent Left_ee, child camera_link, origin xyz=0.02 0.1 -0.1 rpy=-3.1412 0 -1.57079632679
