Commit message: remove moveit package due to major urdf changes

File: src/full_sampling_urdf/urdf/full_sampling_urdf.urdf (robot description, URDF)
Before this commit: robot full_sampling_urdf, 10 links, 9 joints
Links:
- added link link_6, mass 0.14212; collision mesh filename=package://full_sampling_urdf/meshes/link_6.STL; visual mesh filename=package://full_sampling_urdf/meshes/link_6.STL
- link Left_ee: mass 0.12335 -> 0.12478
- link Right_ee: mass 0.12478 -> 0.12335
- link link_1: mass 0.94142 -> 0.68744
- link link_5: mass 0.21482 -> 0.072706
Joints:
- removed joint base_rover
- added joint joint_6: type fixed, parent link_5, child link_6, origin xyz=0 -0.050661 0.25285 rpy=0 0 -0.010445, axis 0 0 0
- joint base_joint: origin xyz=0.248992596226246 0.000708686024747718 0.407000180703943 rpy=0 0 0 -> xyz=0.24899 0.00070869 0.407 rpy=0 0 0
- joint joint_2: limit lower=-3.14 upper=3.14 effort=100 velocity=2 -> lower=0 upper=3.14 effort=100 velocity=2
- joint joint_3: limit lower=-3.14 upper=3.14 effort=50 velocity=4 -> lower=0 upper=6.28 effort=50 velocity=4; origin xyz=0 0.5275 0.1315 rpy=0 0 -1.0681 -> xyz=0 0.5275 0.1315 rpy=0 0 -1.0686
- joint joint_4: axis 0 0 -1 -> -0.031013 0 -0.99952; origin xyz=0 -0.12961 0.10761 rpy=1.5708 0.017046 0 -> xyz=6.8566E-05 -0.12961 0.10761 rpy=-0.50301 1.5354 -2.073
- joint joint_5: origin xyz=0.083 0.0042084 0.10261 rpy=-1.5708 0 -1.5201 -> xyz=-0.0010256 0.083 0.10269 rpy=-1.5692 0.030978 0.050701
- joint joint_lee: origin xyz=-0.03 -0.0028 0.072 rpy=1.5692 0.05065 -0.031058 -> xyz=0.029494 0.048172 -0.18085 rpy=1.5724 -0.050652 3.121; parent link_5 -> link_6
- joint joint_ree: origin xyz=0.03 -0.0028 0.072 rpy=1.5724 -0.05065 3.1105 -> xyz=-0.030503 0.047545 -0.18085 rpy=1.5692 0.050652 -0.020613; parent link_5 -> link_6

Commit message: fix: root link of urdf

File: src/full_sampling_urdf/urdf/full_sampling_urdf.urdf (robot description, URDF)
Before this commit: robot full_sampling_urdf, 11 links, 9 joints
Joints:
- added joint base_rover: type fixed, parent world, child rover, origin xyz=0.0 0.0 0.00001 rpy=0 0 0

Commit message: modfiy joint 2 limits

File: src/full_sampling_urdf/urdf/full_sampling_urdf.urdf (robot description, URDF)
Before this commit: robot full_sampling_urdf, 11 links, 10 joints
Joints:
- joint joint_2: limit lower=0 upper=3.14 effort=100 velocity=2 -> lower=-3.14 upper=0 effort=100 velocity=2

Commit message: modfiy joint 2 limits

File: src/full_sampling_urdf/urdf/full_sampling_urdf.urdf (robot description, URDF)
Before this commit: robot full_sampling_urdf, 11 links, 10 joints
Joints:
- joint joint_2: limit lower=-3.14 upper=0 effort=100 velocity=2 -> lower=-4.7124 upper=0 effort=100 velocity=2

Commit message: modfiy joint 4 limits

File: src/full_sampling_urdf/urdf/full_sampling_urdf.urdf (robot description, URDF)
Before this commit: robot full_sampling_urdf, 11 links, 10 joints
Joints:
- joint joint_4: limit lower=-3.14 upper=3.14 effort=50 velocity=4 -> lower=0 upper=6.28 effort=50 velocity=4

Commit message: modfiy joint 2 axis of rotation and limits

File: src/full_sampling_urdf/urdf/full_sampling_urdf.urdf (robot description, URDF)
Before this commit: robot full_sampling_urdf, 11 links, 10 joints
Joints:
- joint joint_2: axis 0.035393 0 0.99937 -> -0.035393 0 -0.99937; limit lower=-4.7124 upper=0 effort=100 velocity=2 -> lower=0 upper=4.71 effort=100 velocity=2

Commit message: modified joint_6 type to make link_6 recognizable by gazebo

File: src/full_sampling_urdf/urdf/full_sampling_urdf.urdf (robot description, URDF)
Before this commit: robot full_sampling_urdf, 11 links, 10 joints
Joints:
- joint joint_6: axis 0 0 0 -> 0 0 -1; limit (none) -> lower=0 upper=0 effort=10 velocity=0; type fixed -> revolute
