Commit message: changed root link to world

File: src/sampling_rover_with_arm_urdf/urdf/sampling_rover_with_arm_urdf.urdf (robot description, URDF)
Before this commit: robot sampling_rover_with_arm_urdf, 10 links, 9 joints
Links:
- removed link base_footprint
- added link world
Joints:
- joint base_rover: parent base_footprint -> world

Commit message: removed the mimic tag and added transmission tag for joint_lee

File: src/sampling_rover_with_arm_urdf/urdf/sampling_rover_with_arm_urdf.urdf (robot description, URDF)
Before this commit: robot sampling_rover_with_arm_urdf, 10 links, 9 joints
Joints:
- joint joint_lee: mimic joint=joint_ree multiplier=-1.0 offset=0.0 -> (none)
- joint joint_ree: limit lower=0 upper=0.8 effort=15 velocity=0 -> lower=0 upper=0.8 effort=15 velocity=6

Commit message: add teleop mode

File: src/sampling_rover_with_arm_urdf/urdf/sampling_rover_with_arm_urdf.urdf (robot description, URDF)
Before this commit: robot sampling_rover_with_arm_urdf, 10 links, 9 joints
Links:
- added link camera_depth_optical_frame, mass 0.001
- added link camera_link1, mass 0.001; visual box size=0.01 0.01 0.01
- added link camera_link2, mass 0.001; visual box size=0.01 0.01 0.01
Joints:
- added joint camera_depth_optical_joint: type fixed, parent camera_link2, child camera_depth_optical_frame, origin xyz=0 0 0 rpy=-1.57079632679 0 -1.57079632679
- added joint camera_joint1: type fixed, parent Left_ee, child camera_link1, origin xyz=0.02 0.1 -0.1 rpy=-3.1412 0 -1.57079632679
- added joint camera_joint2: type fixed, parent rover, child camera_link2, origin xyz=0 0.3 0.35 rpy=0 0 1.57079632679

Commit message: add IKSolver script

File: src/sampling_rover_with_arm_urdf/urdf/sampling_rover_with_arm_urdf.urdf (robot description, URDF)
Before this commit: robot sampling_rover_with_arm_urdf, 13 links, 12 joints
Joints:
- joint camera_joint1: origin xyz=0.02 0.1 -0.1 rpy=-3.1412 0 -1.57079632679 -> xyz=0.12 0.0 -0.3 rpy=-3.1412 -1.57079632679 0; parent Left_ee -> link_5

Commit message: add IKSolver update

File: src/sampling_rover_with_arm_urdf/urdf/sampling_rover_with_arm_urdf.urdf (robot description, URDF)
Before this commit: robot sampling_rover_with_arm_urdf, 13 links, 12 joints
Joints:
- joint joint_1: limit lower=-3.142 upper=3.142 effort=100 velocity=2 -> lower=-3.142 upper=3.142 effort=100 velocity=1
- joint joint_2: limit lower=-3.142 upper=3.142 effort=100 velocity=2 -> lower=-3.142 upper=3.142 effort=100 velocity=1
- joint joint_3: limit lower=-3.142 upper=3.142 effort=50 velocity=4 -> lower=-3.142 upper=3.142 effort=50 velocity=1
- joint joint_4: limit lower=-3.142 upper=3.142 effort=50 velocity=4 -> lower=-3.142 upper=3.142 effort=50 velocity=1
- joint joint_5: limit lower=-3.142 upper=3.142 effort=50 velocity=4 -> lower=-3.142 upper=3.142 effort=50 velocity=1
- joint joint_lee: limit lower=-0.8 upper=0 effort=15 velocity=6 -> lower=-0.8 upper=0 effort=15 velocity=1
- joint joint_ree: limit lower=0 upper=0.8 effort=15 velocity=6 -> lower=0 upper=0.8 effort=15 velocity=1
