Commit message: added camera plugin

File: movit_full_sampling/urdf/full_sampling_urdf.urdf (robot description, URDF)
Before this commit: robot full_sampling_urdf, 11 links, 10 joints
Links:
- added link camera_depth_optical_frame, mass 0.001
- added link camera_link1, mass 0.001; visual box size=0.01 0.01 0.01
- added link camera_link2, mass 0.001; visual box size=0.01 0.01 0.01
Joints:
- added joint camera_depth_optical_joint: type fixed, parent camera_link2, child camera_depth_optical_frame, origin xyz=0 0 0 rpy=-1.57079632679 0 -1.57079632679
- added joint camera_joint1: type fixed, parent link_5, child camera_link1, origin xyz=0 0.105 0.05 rpy=-1.57079632679 -1.57079632679 0
- added joint camera_joint2: type fixed, parent rover, child camera_link2, origin xyz=0.375 0 0.4 rpy=0 0 0

Commit message: collision in urdf changed

File: movit_full_sampling/urdf/full_sampling_urdf.urdf (robot description, URDF)
Before this commit: robot full_sampling_urdf, 14 links, 13 joints
Links:
- link rover: geometry collision box size=0.6 0.4 0.3; visual mesh filename=package://movit_full_sampling/meshes/rover.STL

Commit message: collision box dimensions

File: movit_full_sampling/urdf/full_sampling_urdf.urdf (robot description, URDF)
Before this commit: robot full_sampling_urdf, 14 links, 13 joints
Links:
- link rover: geometry collision box size=0.9 0.8 0.5; visual box size=0.9 0.8 0.5

Commit message: urdf latest collision changes

File: movit_full_sampling/urdf/full_sampling_urdf.urdf (robot description, URDF)
Before this commit: robot full_sampling_urdf, 14 links, 13 joints
Links:
- link rover: geometry collision box size=0.3 0.25 0.24; collision box size=0.3 0.25 0.24
